File: X9-Backplane.sch (EAGLE design)
At the start: 15 parts

Commit message: silk screen and wiring
Connections:
- net TX_BT: now also U$1G$1.24; no longer U$1G$1.20
Changed lines of the file:
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@@
 <net name="TX_BT" class="0">
-<segment>
-<pinref part="U$1" gate="G$1" pin="20"/>
-<wire x1="373.38" y1="137.16" x2="381" y2="137.16" width="0.1524" layer="91"/>
-<label x="373.38" y="137.16" size="1.778" layer="95"/>
-</segment>
 <segment>
 <pinref part="BT_SIGNAL" gate="G$1" pin="1"/>
@@
 <label x="215.9" y="71.12" size="1.778" layer="95" rot="R90"/>
 </segment>
+<segment>
+<pinref part="U$1" gate="G$1" pin="24"/>
+<wire x1="373.38" y1="142.24" x2="381" y2="142.24" width="0.1524" layer="91"/>
+<label x="373.38" y="142.24" size="1.778" layer="95"/>
+</segment>
 </net>
